Commit message: Add files via upload

File: ARM5.urdf.xacro (robot description, xacro)
@@ -41,5 +41,6 @@
                 <cylinder length="0.1" radius="0.06" />
             </geometry>
-            <material name="blue">    <!-- BLUE had rgba values described in include file -->
+            <material name="blue">
+                <color rgba="0.2 0.2 1 1"/>
             </material>
         </visual>
@@ -50,6 +51,8 @@
             </geometry>
         </collision>
-        <xacro:inertial_cylinder mass="1.5" length="0.1" radius="0.06">
+        <inertial>
             <origin xyz="0 0 0.05" rpy="0 0 0"/>
+            <mass value="1.5" />
+            <inertia ixx="0.001331" ixy="0.0" ixz="0.0" iyy="0.001331" iyz="0.0" izz="0.0027" />
         </inertial>
     </link>
@@ -67,15 +70,19 @@
                 <box size="0.01 0.01 0.01" />
             </geometry>
-            <material name="orange" />
-        </visual>
-        <collision>
-            <origin xyz="0 0.03 0.1" rpy="0 0 0"/>
+            <material name="orange">
+                <color rgba="1 0.3 0.1 1"/>
+            </material>
+        </visual>
+        <collision>
+            <origin xyz="0 0.03 0.105" rpy="0 0 0"/>
             <geometry>
                 <box size="0.01 0.01 0.01" />
             </geometry>
         </collision>
-        <xacro:inertial_box mass="0.05" x="0.01" y="0.01" z="0.01">
-            <origin xyz="0 0.03 0.1" rpy="0 0 0"/>
-        </xacro:inertial_box>
+        <inertial>
+            <origin xyz="0 0.03 0.105" rpy="0 0 0"/>
+            <mass value="0.05" />
+            <inertia ixx="0.0000001" ixy="0.0" ixz="0.0" iyy="0.0000001" iyz="0.0" izz="0.0000001" />
+        </inertial>
     </link>
     <joint name="joint_servo_shaft1" type="revolute">  <!-- DONE, i think -->
@@ -92,15 +99,19 @@
                 <box size="0.04 0.02 0.15" />
             </geometry>
-            <material name="white" />
-        </visual>
-        <collision>
-            <origin xyz="0 0.01 0.075" rpy="0 0 0"/>
-            <geometry>
-                <box size="0.04 0.02 0.15" />
-            </geometry>
-        </collision>
-        <xacro:inertial_box mass="0.1" x="0.04" y="0.02" z="0.15">
-            <origin xyz="0 0.01 0.075" rpy="0 0 0"/>
-        </xacro:inertial_box>
+            <material name="white">
+                <color rgba="1 1 1 1"/>
+            </material>
+        </visual>
+        <collision>
+            <origin xyz="0 0.01 0.075" rpy="0 0 0"/>
+            <geometry>
+                <box size="0.04 0.02 0.15" />
+            </geometry>
+        </collision>
+        <inertial>
+            <origin xyz="0 0.01 0.075" rpy="0 0 0"/>
+            <mass value="0.1" />
+            <inertia ixx="0.0001908" ixy="0.0" ixz="0.0" iyy="0.0002008" iyz="0.0" izz="0.0000167" />
+        </inertial>
     </link>
     <joint name="joint_shaft1_shaft2" type="revolute">  <!-- DONE, i think -->
@@ -117,5 +128,7 @@
                 <box size="0.04 0.02 0.15" />
             </geometry>
-            <material name="white" />
+            <material name="white">
+                <color rgba="1 1 1 1"/>
+            </material>
         </visual>
         <collision>
@@ -125,7 +138,9 @@
             </geometry>
         </collision>
-        <xacro:inertial_box mass="0.1" x="0.04" y="0.02" z="0.15">
+        <inertial>
             <origin xyz="0 -0.01 0.075" rpy="0 0 0"/>
-        </xacro:inertial_box>
+            <mass value="0.1" />
+            <inertia ixx="0.0001908" ixy="0.0" ixz="0.0" iyy="0.0002008" iyz="0.0" izz="0.0000167" />
+        </inertial>
     </link>
     <joint name="joint_shaft2_shaft3" type="revolute">  <!-- DONE, i think -->
@@ -142,15 +157,19 @@
                 <box size="0.04 0.02 0.15" />
             </geometry>
-            <material name="white" />
-        </visual>
-        <collision>
-            <origin xyz="0 0.01 0.075" rpy="0 0 0"/>
-            <geometry>
-                <box size="0.04 0.02 0.15" />
-            </geometry>
-        </collision>
-        <xacro:inertial_box mass="0.1" x="0.04" y="0.02" z="0.15">
-            <origin xyz="0 0.01 0.075" rpy="0 0 0"/>
-        </xacro:inertial_box>
+            <material name="white">
+                <color rgba="1 1 1 1"/>
+            </material>
+        </visual>
+        <collision>
+            <origin xyz="0 0.01 0.075" rpy="0 0 0"/>
+            <geometry>
+                <box size="0.04 0.02 0.15" />
+            </geometry>
+        </collision>
+        <inertial>
+            <origin xyz="0 0.01 0.075" rpy="0 0 0"/>
+            <mass value="0.1" />
+            <inertia ixx="0.0001908" ixy="0.0" ixz="0.0" iyy="0.0002008" iyz="0.0" izz="0.0000167" />
+        </inertial>
     </link>
     <joint name="joint_shaft3_hand" type="revolute">  <!-- DONE, i think -->
@@ -161,5 +180,5 @@
         <limit lower="${-pi/2}" upper="${pi/2}" velocity="100" effort="100"/> <!-- what do I put in effort and velocity again? -->
     </joint>
-    <link name="hand_link">
+    <link name="hand_link">  <!-- DONE, i think -->
         <visual>
             <origin xyz="0 -0.02 0" rpy="0 0 0"/>
@@ -167,5 +186,7 @@
                 <box size="0.04 0.04 0.04" />
             </geometry>
-            <material name="orange" />
+            <material name="orange">
+                <color rgba="1 0.3 0.1 1"/>
+            </material>
         </visual>
         <visual>
@@ -174,5 +195,7 @@
                 <box size="0.04 0.12 0.04" />
             </geometry>
-            <material name="orange" />
+            <material name="orange">
+                <color rgba="1 0.3 0.1 1"/>
+            </material>
         </visual>
         <collision>
@@ -182,8 +205,10 @@
             </geometry>
         </collision>
-        <xacro:inertial_box mass="1" x="0.04" y="0.12" z="0.08">
+        <inertial>
             <origin xyz="0 -0.02 0.02" rpy="0 0 0"/>
-        </xacro:inertial_box>
-    </link>
-    <xacro:include filename="example_gazebo.xacro" />
+            <mass value="1" />
+            <inertia ixx="0.001733" ixy="0.0" ixz="0.0" iyy="0.0006667" iyz="0.0" izz="0.001333" />
+        </inertial>
+    </link>
+    <!-- <xacro:include filename="example_gazebo.xacro" /> -->
 </robot>

Commit message: Add files via upload

File: ARM5.urdf.xacro (robot description, xacro)
@@ -1,28 +1,5 @@
 <?xml version="1.0"?>
 <robot xmlns:xacro="http://www.ros.org/wiki/xacro"  name="robot">
-    <!-- This is an example of a URDF. -->
-    <!-- As we move through the file, new things to note will be pointed out. -->
-    <!-- It's not meant an example of GOOD design, but an example of some of the various features of URDF/xacro. -->
-    <!-- <xacro:include filename="ARM5_include.xacro" />   -->
-    <!-- ROBOT STRUCTURE -->
-    <!-- world -->
-    <!-- base_joint (fixed) -->
-    <!-- base_link (cylinder) -->
-    <!-- joint_base_servo (revolute in Z) [motor1]-->
-    <!-- servo_link (small box) -->
-    <!-- joint_servo_shaft1 (revolute in Y) [motor2]-->
-    <!-- shaft1_link (rectangular box) -->
-    <!-- joint_shaft1_shaft2 (revolute in Y) [motor3]-->
-    <!-- shaft2_link (rectangular box) -->
-    <!-- joint_shaft2_shaft3 (revolute in Y) [motor4]-->
-    <!-- shaft3_link (rectangular box) -->
-    <!-- joint_shaft3_hand (revolute in Y) [motor5]-->
-    <!-- hand_link (god fucking knows) -->
-    <!-- how to include gripper? maybe theres something like there is for camera -->
-    <!-- shafts will have a default size x=0.04 y=0.02 z=0.15 -->
-    <!-- This first link called "world" is empty -->
     <link name="world"></link>
-    <!-- A simple fixed joint from our empty world link, to our base. -->
-    <!-- The base origin is não offset from the world origin. -->
     <joint name="base_joint" type="fixed">
         <origin xyz="0 0 0" rpy="0 0 0"/>
@@ -30,10 +7,5 @@
         <child link="base_link"/>
     </joint>
-    <!-- base_link is a large rectangular plate. Some things to note: -->
-    <!-- - We set the visual origin Z to half the box height, so that the link origin sits at the bottom of the box -->
-    <!-- - We set the collision to be identical to the visual -->
-    <!-- - We specified the colour manually (but still need to enter a name) -->
-    <!-- - We specified all the inertial parameters manually -->
-    <link name="base_link">   <!-- DONE, i think -->
+    <link name="base_link">
         <visual>
             <origin xyz="0 0 0.05" rpy="0 0 0"/>
@@ -57,12 +29,12 @@
         </inertial>
     </link>
-    <joint name="joint_base_servo" type="revolute"> <!-- DONE, i think -->
+    <joint name="joint_base_servo" type="revolute">
         <origin xyz="0 0 0.05" rpy="0 0 0"/>
         <parent link="base_link"/>
         <child link="servo_link"/>
         <axis xyz="0 0 1"/>
-        <limit lower="${-pi/2}" upper="${pi/2}" velocity="100" effort="100"/> <!-- what do I put in effort and velocity again? -->
+        <limit lower="${-pi/2}" upper="${pi/2}" velocity="100" effort="100"/>
     </joint>
-    <link name="servo_link"> <!-- DONE, i think -->
+    <link name="servo_link">
         <visual>
             <origin xyz="0 0.03 0.105" rpy="0 0 0"/>
@@ -86,12 +58,12 @@
         </inertial>
     </link>
-    <joint name="joint_servo_shaft1" type="revolute">  <!-- DONE, i think -->
+    <joint name="joint_servo_shaft1" type="revolute">
         <origin xyz="0 -0.05 0" rpy="0 0 0"/>
         <parent link="servo_link"/>
         <child link="shaft1_link"/>
         <axis xyz="0 1 0"/>
-        <limit lower="${-pi/2}" upper="${pi/2}" velocity="100" effort="100"/> <!-- what do I put in effort and velocity again? -->
+        <limit lower="${-pi/2}" upper="${pi/2}" velocity="100" effort="100"/>
     </joint>
-    <link name="shaft1_link">   <!-- DONE, i think -->
+    <link name="shaft1_link">
         <visual>
             <origin xyz="0 0.01 0.075" rpy="0 0 0"/>
@@ -115,12 +87,12 @@
         </inertial>
     </link>
-    <joint name="joint_shaft1_shaft2" type="revolute">  <!-- DONE, i think -->
-        <origin xyz="0 -0.01 0.075" rpy="0 0 0"/>
+    <joint name="joint_shaft1_shaft2" type="revolute">
+        <origin xyz="0 -0.01 0.15" rpy="0 0 0"/>
         <parent link="shaft1_link"/>
         <child link="shaft2_link"/>
         <axis xyz="0 1 0"/>
-        <limit lower="${-pi/2}" upper="${pi/2}" velocity="100" effort="100"/> <!-- what do I put in effort and velocity again? -->
+        <limit lower="${-pi/2}" upper="${pi/2}" velocity="100" effort="100"/>
     </joint>
-    <link name="shaft2_link">   <!-- DONE, i think -->
+    <link name="shaft2_link">
         <visual>
             <origin xyz="0 -0.01 0.075" rpy="0 0 0"/>
@@ -144,12 +116,12 @@
         </inertial>
     </link>
-    <joint name="joint_shaft2_shaft3" type="revolute">  <!-- DONE, i think -->
-        <origin xyz="0 0.01 0.075" rpy="0 0 0"/>
+    <joint name="joint_shaft2_shaft3" type="revolute">
+        <origin xyz="0 0.01 0.15" rpy="0 0 0"/>
         <parent link="shaft2_link"/>
         <child link="shaft3_link"/>
         <axis xyz="0 1 0"/>
-        <limit lower="${-pi/2}" upper="${pi/2}" velocity="100" effort="100"/> <!-- what do I put in effort and velocity again? -->
+        <limit lower="${-pi/2}" upper="${pi/2}" velocity="100" effort="100"/>
     </joint>
-    <link name="shaft3_link">   <!-- DONE, i think -->
+    <link name="shaft3_link">
         <visual>
             <origin xyz="0 0.01 0.075" rpy="0 0 0"/>
@@ -174,11 +146,11 @@
     </link>
     <joint name="joint_shaft3_hand" type="revolute">  <!-- DONE, i think -->
-        <origin xyz="0 -0.01 0.075" rpy="0 0 0"/>
+        <origin xyz="0 -0.01 0.15" rpy="0 0 0"/>
         <parent link="shaft3_link"/>
         <child link="hand_link"/>
         <axis xyz="0 1 0"/>
-        <limit lower="${-pi/2}" upper="${pi/2}" velocity="100" effort="100"/> <!-- what do I put in effort and velocity again? -->
+        <limit lower="${-pi/2}" upper="${pi/2}" velocity="100" effort="100"/>
     </joint>
-    <link name="hand_link">  <!-- DONE, i think -->
+    <link name="hand_link">
         <visual>
             <origin xyz="0 -0.02 0" rpy="0 0 0"/>
@@ -211,4 +183,3 @@
         </inertial>
     </link>
-    <!-- <xacro:include filename="example_gazebo.xacro" /> -->
 </robot>
