Commit message: Add files via upload

File: ARM5full.urdf.xacro (robot description, xacro)
@@ -192,5 +192,5 @@
     <link name="leftfinger_link">
         <visual>
-            <origin xyz="0 0.0 0.04" rpy="0 0 0"/>
+            <origin xyz="0 0.0 0.08" rpy="0 0 0"/>
             <geometry>
                 <box size="0.04 0.03 0.08" />
@@ -201,11 +201,11 @@
         </visual>
         <collision>
-            <origin xyz="0 0.0 0.04" rpy="0 0 0"/>
-            <geometry>
-                <box size="0.04 0.03 0.08" />
-            </geometry>
-        </collision>
-        <inertial>
-            <origin xyz="0 0.0 0.04" rpy="0 0 0"/>
+            <origin xyz="0 0.0 0.08" rpy="0 0 0"/>
+            <geometry>
+                <box size="0.04 0.03 0.08" />
+            </geometry>
+        </collision>
+        <inertial>
+            <origin xyz="0 0.0 0.08" rpy="0 0 0"/>
             <mass value="0.1" />
             <inertia ixx="0.000060833" ixy="0.0" ixz="0.0" iyy="0.00006666" iyz="0.0" izz="0.000020833" />
@@ -221,5 +221,5 @@
     <link name="rightfinger_link">
         <visual>
-            <origin xyz="0 0.0 0.04" rpy="0 0 0"/>
+            <origin xyz="0 0.0 0.08" rpy="0 0 0"/>
             <geometry>
                 <box size="0.04 0.03 0.08" />
@@ -230,11 +230,11 @@
         </visual>
         <collision>
-            <origin xyz="0 0.0 0.04" rpy="0 0 0"/>
-            <geometry>
-                <box size="0.04 0.03 0.08" />
-            </geometry>
-        </collision>
-        <inertial>
-            <origin xyz="0 0.0 0.04" rpy="0 0 0"/>
+            <origin xyz="0 0.0 0.08" rpy="0 0 0"/>
+            <geometry>
+                <box size="0.04 0.03 0.08" />
+            </geometry>
+        </collision>
+        <inertial>
+            <origin xyz="0 0.0 0.08" rpy="0 0 0"/>
             <mass value="0.1" />
             <inertia ixx="0.000060833" ixy="0.0" ixz="0.0" iyy="0.00006666" iyz="0.0" izz="0.000020833" />
